Commit message: fix:mathtools

File: armcontrol/xacro/arm.xacro (robot description, xacro)
@@ -8,12 +8,5 @@
   <xacro:property name="base_link_height" value="0.079989"/>
   <xacro:property name="pi" value="3.14159265353846"/>
-<xacro:property name="link" value="0.10001"/>
-  <joint name="arm_base_joint" type="fixed">
-    <origin
-      xyz="0 0 0"
-      rpy="0 0 0" />
-    <parent link="arm_base_link" />
-    <child link="arm_link_1" />
-  </joint>
+  <xacro:property name="link" value="0.10001"/>
   <link
     name="arm_base_link">
@@ -74,5 +67,5 @@
     <visual>
       <origin
-        xyz="0 0 ${-3.3733E-07-0.10001}"
+        xyz="0 0 -0.10001"
         rpy="${pi/2} 0 ${-pi/2}" />
       <geometry>
@@ -88,6 +81,6 @@
     <collision>
       <origin
-        xyz="0 0 0"
-        rpy="0 0 0" />
+        xyz="0 0 -0.10001"
+        rpy="${pi/2} 0 ${-pi/2}" />
       <geometry>
         <mesh
@@ -117,10 +110,9 @@
       friction="${motor_fric}" />
   </joint>
-<!-- xyz="4.1945E-10 0.2726 -9.6287E-12" -->
   <link
     name="arm_link_2">
     <inertial>
       <origin
-        xyz="0 0 0"
+        xyz="4.1945E-10 0.2726 -9.6287E-12"
         rpy="0 0 0" />
       <mass
@@ -151,5 +143,5 @@
       <origin
         xyz="0 0 0"
-        rpy="0 0 0" />
+        rpy="0 ${pi/2} ${-pi/2}" />
       <geometry>
         <mesh
@@ -179,10 +171,9 @@
       friction="${motor_fric}" />
   </joint>
-<!--  xyz="-3.4632E-18 0.28121 1.1102E-16" "  -->
   <link
     name="arm_link_3">
     <inertial>
       <origin
-        xyz="0 0 0"
+         xyz="-3.4632E-18 0.28121 1.1102E-16"
         rpy="0 0 0" />
       <mass
@@ -213,5 +204,5 @@
       <origin
         xyz="0 0 0"
-        rpy="0 0 0" />
+        rpy="0 ${pi/2} ${-pi/2}" />
       <geometry>
         <mesh
@@ -241,10 +232,10 @@
       friction="${motor_fric}" />
   </joint>
-<!--   xyz="1.9004E-18 0.049824 0 "  -->
+<!--     -->
   <link
     name="arm_link_4">
     <inertial>
       <origin
-        xyz="0 0 0 "
+        xyz="1.9004E-18 0.049824 0 "
         rpy="0 0 0" />
       <mass
@@ -275,5 +266,5 @@
       <origin
         xyz="0 0 0"
-        rpy="0 0 0" />
+        rpy="0 0 1.5707" />
       <geometry>
         <mesh
@@ -303,10 +294,9 @@
       friction="${motor_fric}" />
   </joint>
-<!--   xyz="-1.1102E-16 -0.014377 -2.4389E-17"   -->
   <link
     name="arm_link_5">
     <inertial>
       <origin
-        xyz="0 0 0"
+         xyz="-1.1102E-16 -0.014377 -2.4389E-17"
         rpy="0 0 0" />
       <mass
@@ -336,6 +326,6 @@
     <collision>
       <origin
-        xyz="0 0 0"
-        rpy="0 0 0" />
+         xyz="0 0 0"
+        rpy="0 0 1.5707" />
       <geometry>
         <mesh
@@ -397,6 +387,6 @@
     <collision>
       <origin
-        xyz="0 0 0"
-        rpy="0 0 0" />
+         xyz="0 0 0"
+        rpy="0 0 1.5707" />
       <geometry>
         <mesh
@@ -466,6 +456,6 @@
     <collision>
       <origin
-        xyz="0 0 0"
-        rpy="0 0 0" />
+         xyz="0 0 0"
+        rpy="-1.5707 0 0"  />
       <geometry>
         <mesh
@@ -536,5 +526,5 @@
       <origin
         xyz="0 0 0"
-        rpy="0 0 0" />
+        rpy="1.5707 0 0" />
       <geometry>
         <mesh

Commit message: fix error

File: armcontrol/xacro/arm.xacro (robot description, xacro)
@@ -8,5 +8,12 @@
   <xacro:property name="base_link_height" value="0.079989"/>
   <xacro:property name="pi" value="3.14159265353846"/>
-  <xacro:property name="link" value="0.10001"/>
+<xacro:property name="link" value="0.10001"/>
+  <joint name="arm_base_joint" type="fixed">
+    <origin
+      xyz="0 0 0"
+      rpy="0 0 0" />
+    <parent link="arm_base_link" />
+    <child link="arm_link_1" />
+  </joint>
   <link
     name="arm_base_link">
@@ -67,5 +74,5 @@
     <visual>
       <origin
-        xyz="0 0 -0.10001"
+        xyz="0 0 ${-3.3733E-07-0.10001}"
         rpy="${pi/2} 0 ${-pi/2}" />
       <geometry>
@@ -81,6 +88,6 @@
     <collision>
       <origin
-        xyz="0 0 -0.10001"
-        rpy="${pi/2} 0 ${-pi/2}" />
+        xyz="0 0 0"
+        rpy="0 0 0" />
       <geometry>
         <mesh
@@ -110,9 +117,10 @@
       friction="${motor_fric}" />
   </joint>
+<!-- xyz="4.1945E-10 0.2726 -9.6287E-12" -->
   <link
     name="arm_link_2">
     <inertial>
       <origin
-        xyz="4.1945E-10 0.2726 -9.6287E-12"
+        xyz="0 0 0"
         rpy="0 0 0" />
       <mass
@@ -143,5 +151,5 @@
       <origin
         xyz="0 0 0"
-        rpy="0 ${pi/2} ${-pi/2}" />
+        rpy="0 0 0" />
       <geometry>
         <mesh
@@ -171,9 +179,10 @@
       friction="${motor_fric}" />
   </joint>
+<!--  xyz="-3.4632E-18 0.28121 1.1102E-16" "  -->
   <link
     name="arm_link_3">
     <inertial>
       <origin
-         xyz="-3.4632E-18 0.28121 1.1102E-16"
+        xyz="0 0 0"
         rpy="0 0 0" />
       <mass
@@ -204,5 +213,5 @@
       <origin
         xyz="0 0 0"
-        rpy="0 ${pi/2} ${-pi/2}" />
+        rpy="0 0 0" />
       <geometry>
         <mesh
@@ -232,10 +241,10 @@
       friction="${motor_fric}" />
   </joint>
-<!--     -->
+<!--   xyz="1.9004E-18 0.049824 0 "  -->
   <link
     name="arm_link_4">
     <inertial>
       <origin
-        xyz="1.9004E-18 0.049824 0 "
+        xyz="0 0 0 "
         rpy="0 0 0" />
       <mass
@@ -266,5 +275,5 @@
       <origin
         xyz="0 0 0"
-        rpy="0 0 1.5707" />
+        rpy="0 0 0" />
       <geometry>
         <mesh
@@ -294,9 +303,10 @@
       friction="${motor_fric}" />
   </joint>
+<!--   xyz="-1.1102E-16 -0.014377 -2.4389E-17"   -->
   <link
     name="arm_link_5">
     <inertial>
       <origin
-         xyz="-1.1102E-16 -0.014377 -2.4389E-17"
+        xyz="0 0 0"
         rpy="0 0 0" />
       <mass
@@ -326,6 +336,6 @@
     <collision>
       <origin
-         xyz="0 0 0"
-        rpy="0 0 1.5707" />
+        xyz="0 0 0"
+        rpy="0 0 0" />
       <geometry>
         <mesh
@@ -387,6 +397,6 @@
     <collision>
       <origin
-         xyz="0 0 0"
-        rpy="0 0 1.5707" />
+        xyz="0 0 0"
+        rpy="0 0 0" />
       <geometry>
         <mesh
@@ -456,6 +466,6 @@
     <collision>
       <origin
-         xyz="0 0 0"
-        rpy="-1.5707 0 0"  />
+        xyz="0 0 0"
+        rpy="0 0 0" />
       <geometry>
         <mesh
@@ -526,5 +536,5 @@
       <origin
         xyz="0 0 0"
-        rpy="1.5707 0 0" />
+        rpy="0 0 0" />
       <geometry>
         <mesh
